File: hardware/eagle/candy-avb.sch (EAGLE design)
At the start: 161 parts, among them IC1 TPS2115ASON, IC11 ADAU1761ORIGINAL, IC2 TPS63061, IC3 10M08SCUBGA169, IC4 CP2012N-20, IC5 ADAU1761ORIGINAL, IC6 DP83848, IC7 MIC5219-3.3YM5, IC9 TXB0108ZXYR, J2 TE_MODULAR_JACK_1734577-1TOP, J4 2X6 FEMALE, X1 48MHz, X2 USBi, X3 USB Blaster

Commit message: Release v0.3.
Parts:
- added TP10, TP11, TP12, TP13, TP14, TP15, TP16, TP17, TP18, TP19, TP2, TP20, TP21, TP3, TP4, TP5, TP6, TP7, TP8, TP9, UART_CTS, UART_RTS, UART_RX, UART_TX: TPB1,27, testpad:TPB1,27
Connections:
- new net CLK2MAC: IC6.CLK2MAC, TP21.TP
- new net E3: IC3G$1.E3, J4.14
- new net E4: IC3G$1.E4, J4.4
- new net LED_SPD: IC6.LED_SPD, TP20.TP
- new net RX_DV: IC6.RX_DV, TP19.TP
- net COL: now also TP5.TP
- net CRS: now also TP3.TP
- net EINT: now also TP16.TP
- net L2: no longer J4.4
- net LS_A2: now also IC3G$7.A2; no longer IC3G$7.B3
- net LS_A3: now also IC3G$7.B3; no longer IC3G$7.A2
- net MDC: now also TP18.TP
- net MDIO: now also TP17.TP
- net N3: no longer J4.14
- net RXD0: now also TP6.TP
- net RXD1: now also TP7.TP
- net RXD2: now also TP8.TP
- net RXD3: now also TP9.TP
- net RX_CLK: now also TP2.TP
- net RX_ER: now also TP4.TP
- net TXD0: now also TP12.TP
- net TXD1: now also TP13.TP
- net TXD2: now also TP14.TP
- net TXD3: now also TP15.TP
- net TXEN: now also TP11.TP
- net TX_CLK: now also TP10.TP
- net UART_CTS: now also UART_CTS.TP
- net UART_RTS: now also UART_RTS.TP
- net UART_RX: now also UART_RX.TP
- net UART_TX: now also UART_TX.TP
Other:
- moved on the sheet: C23, R44

Commit message: Release v0.4.
Parts:
- renumbered USER_SW to RESET_SW
Connections:
- net BITCLOCK: now also IC3G$4.M5; no longer IC3G$4.N5
- net COL: now also IC3G$4.N11-VREFB3NO; no longer IC3G$4.L10
- net CRS: now also IC3G$4.N12; no longer IC3G$4.M11
- net DATA_IN: now also IC3G$4.N5; no longer IC3G$4.M5
- net DATA_OUT: now also IC3G$4.K6; no longer IC3G$4.N6
- net DATA_OUT_2: now also IC3G$4.L5; no longer IC3G$4.N4
- net LRCLOCK: now also IC3G$4.N4; no longer IC3G$4.L5
- net RXD0: now also IC3G$4.L10; no longer IC3G$4.N11-VREFB3NO
- net RXD1: now also IC3G$4.N10; no longer IC3G$4.M10
- net RXD2: now also IC3G$4.M10; no longer IC3G$4.N10
- net RXD3: now also IC3G$4.N9; no longer IC3G$4.M9
- net RX_CLK: now also IC3G$4.L11; no longer IC3G$4.M12
- net RX_DV: now also IC3G$4.M12
- net RX_ER: now also IC3G$4.M11; no longer IC3G$4.N12
- net TXD0: now also IC3G$4.M8; no longer IC3G$4.N8
- net TXD1: now also IC3G$4.N7; no longer IC3G$4.M7
- net TXD2: now also IC3G$4.M7; no longer IC3G$4.N7
- net TXD3: now also IC3G$4.N6; no longer IC3G$4.K6
- net TXEN: now also IC3G$4.N8; no longer IC3G$4.M8
- net TX_CLK: now also IC3G$4.M9; no longer IC3G$4.N9

Commit message: Release v0.5
Change C26 from 47uF to 22uF x3.
Change C1 from 47uF to 10uF x2.
Change L1 package size.
Create GND plane on top layer.
Parts:
- added C10, C6: 22uF, tkrworks:C-EUC0805
- added C11: 10uF, tkrworks:C-EUC0805
- added R19: 33, tkrworks:RESISTOR0402-RES
- C1: value 47uF -> 10uF; device tkrworks:C-EUC1210 -> tkrworks:C-EUC0805
- C14: value 10uF -> 10uF tant
- C26: value 47uF -> 22uF; device tkrworks:C-EUC1210 -> tkrworks:C-EUC0805
- L1: device tkrworks:L_1210 -> tkrworks:L_4240
Connections:
- new net N$21: IC6.RX_DV, R19.2
- net BAT: now also C10.1, C6.1
- net GND: now also C10.2, C11.2, C6.2
- net RX_DV: now also R19.1; no longer IC6.RX_DV
- net VIN: now also C11.1
Other:
- moved on the sheet: BITCLOCK1, C24, C57, C58, C64, C65, C66, C67, C68, C69, C70, C71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

Commit message: Release v0.6
Add the power switch MIC2005A to reset the ADAU1772.
Parts:
- added C28: 1uF, tkrworks:C-EUC0603
- added IC10: MIC2005A, tkrworks:MIC20XXSOT23-5
- added R20: 10k, tkrworks:RESISTOR0402-RES
Connections:
- new net EN1: C72.1, IC7.EN, R59.2
- new net VOUT: C20.1, C56.1, C58.1, C59.1, C60.1, C61.2, C62.2, C63.2, C64.1, C65.1, C66.1, C67.2, C68.2, C69.2, IC10.5.VOUT, IC11.AVDD, IC11.AVDD_2, IC11.DVDOUT, IC11.IOVDD, IC5.AVDD, IC5.AVDD_2, IC5.DVDOUT, IC5.IOVDD
- net BRD_RESET: now also IC10.3.ENA, IC3G$3.L1-VREFB2NO, R20.2; no longer C72.1, IC7.EN, R59.2
- net GND: now also C28.2, IC10.2.GND
- net VDD: now also C28.1, IC10.1.VIN, R20.1; no longer C20.1, C56.1, C58.1, C59.1, C60.1, C61.2, C62.2, C63.2, C64.1, C65.1, C66.1, C67.2, C68.2, C69.2, IC11.AVDD, IC11.AVDD_2, IC11.DVDOUT, IC11.IOVDD, IC5.AVDD, IC5.AVDD_2, IC5.DVDOUT, IC5.IOVDD
